File: STM32F4_REV2/STM32F4_REV2.kicad_pcb (KiCad board)
At the start: 4 copper layers, 56.8 x 57.5 mm, 50 parts, among them J1 Screw_Terminal_01x02, J2 SWD, J3 Conn_01x04, J4 Conn_01x04, J5 USB_B_Micro, Q1 AO3401A, SW1 SW_SPDT, U1 STM32F405RGT6, U3 USBLC6-2SC6, Y1 16MHz

Commit message: Finished routing
Parts:
- moved H2 5.34 mm to (80.0, 89.7)
- moved H1 4.81 mm to (80.9, 43.4)
- moved J5 4.50 mm to (83.2, 57.8)
- moved U3 4.50 mm to (76.2, 58.1)
- moved R10 1.32 mm to (51.8, 54.4)
- moved R9 1.32 mm to (54.2, 54.4)
- moved D4 0.82 mm to (72.9, 40.4)
- moved R11 0.81 mm to (73.0, 43.1)
- moved J2 0.81 mm to (64.5, 42.6)
- moved C13 0.55 mm to (71.3, 75.0)
- moved R8 0.15 mm to (78.0, 82.1)
- moved R3 0.12 mm to (45.5, 72.1)
- moved R7 0.08 mm to (76.2, 82.1)
- moved C15 0.05 mm to (65.8, 85.8)
Routing:
- net GND: track 0.00 -> 68.2 mm, vias 0 -> 42
- net +3.3V: track 0.00 -> 48.8 mm, vias 0 -> 24
- net NRST: track 0.00 -> 36.3 mm, vias 0 -> 2
- net SWO: track 0.00 -> 24.5 mm
- net SWDIO: track 0.00 -> 23.9 mm, vias 0 -> 2
- net USART3_TX: track 0.00 -> 20.1 mm
- net USART3_RX: track 0.00 -> 19.8 mm
- net SWCLK: track 0.00 -> 17.7 mm
- net USB_D-: track 0.00 -> 17.7 mm
- net USB_D+: track 0.00 -> 17.7 mm
- net I2C1_SDA: track 0.00 -> 15.7 mm
- net +5V: track 0.00 -> 15.5 mm
- net I2C1_SCL: track 0.00 -> 15.0 mm
- net BOOT0: track 0.00 -> 13.9 mm
- net BUCK_IN: track 0.00 -> 11.9 mm
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- added copper zone on In2.Cu, net +3.3V
- added copper zone on In1.Cu, net GND
Other:
- board size 56.8 x 57.5 mm -> 52.5 x 57.5 mm
- board text added: "3V3"
- board text added: "BOOT"
- board text added: "I2C"
- board text added: "POWER"
- board text added: "STATUS"
- board text added: "SWD"
- board text added: "UART"
- board text added: "USB"
